Commit message: Test for tuesday

File: lego_robot_description/urdf/lego_bot.xacro (robot description, xacro)
@@ -23,4 +23,10 @@
     <origin xyz="0.0 0.0 0.0" rpy="0.0 0.0 0.0" />
   </joint>
+  <link name="tool0_controller"/>
+  <joint name="base-tool0_controller_floating_joint" type="floating">
+    <origin xyz="0 0 0" rpy="0 0 0"/>
+    <parent link="base"/>
+    <child link="tool0_controller"/>
+  </joint>
   <!-- Gripper -->
   <xacro:include filename="$(find lego_robot_description)/urdf/gripper.xacro" />

Commit message: all works

File: lego_robot_description/urdf/lego_bot.xacro (robot description, xacro)
@@ -14,5 +14,5 @@
     wrist_1_lower_limit="${-pi}" wrist_1_upper_limit="${pi}"
     wrist_2_lower_limit="${-pi}" wrist_2_upper_limit="${pi}"
-    wrist_3_lower_limit="${-pi}" wrist_3_upper_limit="${pi}"
+    wrist_3_lower_limit="0" wrist_3_upper_limit="${2 * pi}"
     transmission_hw_interface="$(arg transmission_hw_interface)"
   />
@@ -24,5 +24,5 @@
   </joint>
   <link name="tool0_controller"/>
-  <joint name="base-tool0_controller_floating_joint" type="floating">
+  <joint name="base_tool0_controller_floating_joint" type="fixed">
     <origin xyz="0 0 0" rpy="0 0 0"/>
     <parent link="base"/>
@@ -34,5 +34,5 @@
     <parent link="ee_link" />
     <child link = "gripper_body" />
-    <origin xyz="0.0 0.0 0.0" rpy="0 0.0 1.57079632679" />
+    <origin xyz="0.0 0.0 0.0" rpy="0.0 -1.57079632679 1.57079632679" />
   </joint>
   <!-- Realsense Cam -->

Commit message: added tf avg for worldframe

File: lego_robot_description/urdf/lego_bot.xacro (robot description, xacro)
@@ -34,5 +34,11 @@
     <parent link="ee_link" />
     <child link = "gripper_body" />
-    <origin xyz="0.0 0.0 0.0" rpy="0.0 -1.57079632679 1.57079632679" />
+    <origin xyz="0.06 0.0 0.0" rpy="0.0 -1.57079632679 1.57079632679" />
+  </joint>
+  <link name="TCP"/>
+  <joint name="set_tcp" type="fixed">
+    <parent link="gripper_body" />
+    <child link = "TCP" />
+    <origin xyz="0.0 -0.26 0.0" rpy="0.0 3.14159265359 3.14159265359" />
   </joint>
   <!-- Realsense Cam -->

Commit message: fml

File: lego_robot_description/urdf/lego_bot.xacro (robot description, xacro)
@@ -2,25 +2,18 @@
 <robot xmlns:xacro="http://wiki.ros.org/xacro"
        name="ur5" >
-  <xacro:arg name="transmission_hw_interface" default="hardware_interface/PositionJointInterface"/>
-  <!-- common stuff -->
-  <xacro:include filename="$(find ur_description)/urdf/common.gazebo.xacro" />
-  <!-- ur5 -->
-  <xacro:include filename="$(find ur_description)/urdf/ur5.urdf.xacro" />
-  <!-- arm -->
-  <xacro:ur5_robot prefix="" joint_limited="true"
-    shoulder_pan_lower_limit="${-pi}" shoulder_pan_upper_limit="${pi}"
-    shoulder_lift_lower_limit="${-pi}" shoulder_lift_upper_limit="${pi}"
-    elbow_joint_lower_limit="${-pi}" elbow_joint_upper_limit="${pi}"
-    wrist_1_lower_limit="${-pi}" wrist_1_upper_limit="${pi}"
-    wrist_2_lower_limit="${-pi}" wrist_2_upper_limit="${pi}"
-    wrist_3_lower_limit="0" wrist_3_upper_limit="${2 * pi}"
-    transmission_hw_interface="$(arg transmission_hw_interface)"
-  />
-  <link name="world" />
-  <joint name="world_joint" type="fixed">
-    <parent link="world" />
-    <child link = "table" />
-    <origin xyz="0.0 0.0 0.0" rpy="0.0 0.0 0.0" />
-  </joint>
+   <xacro:arg name="transmission_hw_interface" default="hardware_interface/PositionJointInterface"/>
+   <!-- common stuff -->
+   <xacro:include filename="$(find ur_description)/urdf/common.gazebo.xacro"/>
+   <!-- ur5 -->
+   <xacro:include filename="$(find ur_description)/urdf/ur5.urdf.xacro"/>
+   <!-- arm -->
+   <xacro:arg name="kinematics_config" default="$(find ur_description)/config/ur5_default.yaml"/>
+   <xacro:ur5_robot prefix="" joint_limited="true" shoulder_pan_lower_limit="${-pi}" shoulder_pan_upper_limit="${pi}" shoulder_lift_lower_limit="${-pi}" shoulder_lift_upper_limit="${pi}" elbow_joint_lower_limit="${-pi}" elbow_joint_upper_limit="${pi}" wrist_1_lower_limit="${-pi}" wrist_1_upper_limit="${pi}" wrist_2_lower_limit="${-pi}" wrist_2_upper_limit="${pi}" wrist_3_lower_limit="${-pi}" wrist_3_upper_limit="${pi}" transmission_hw_interface="$(arg transmission_hw_interface)" kinematics_file="${load_yaml('$(arg kinematics_config)')}"/>
+   <link name="world"/>
+   <joint name="world_joint" type="fixed">
+   <parent link="world"/>
+   <child link="base_link"/>
+   <origin xyz="0.0 0.0 0.0" rpy="0.0 0.0 0.0"/>
+   </joint>
   <link name="tool0_controller"/>
   <joint name="base_tool0_controller_floating_joint" type="fixed">
@@ -45,5 +38,5 @@
   <xacro:include filename="$(find realsense2_description)/urdf/_d435.urdf.xacro" />
   <sensor_d435 parent="gripper_body">
-    <origin xyz="0  -0.115 0.039" rpy="0 0 -1.57079632679"/>
+    <origin xyz="0  -0.1157 0.03799" rpy="0 0 -1.57079632679"/>
   </sensor_d435>
     <!-- Table -->
@@ -51,5 +44,5 @@
   <joint name="table_mount_robot" type="fixed">
     <parent link="table" />
-    <child link = "base_link" />
+    <child link = "world" />
     <origin xyz="0.0 0.0 0.0" rpy="0.0 0.0 0.0" />
   </joint>

Commit message: updated for new driver

File: lego_robot_description/urdf/lego_bot.xacro (robot description, xacro)
@@ -3,17 +3,17 @@
        name="ur5" >
    <xacro:arg name="transmission_hw_interface" default="hardware_interface/PositionJointInterface"/>
-   <!-- common stuff -->
-   <xacro:include filename="$(find ur_description)/urdf/common.gazebo.xacro"/>
-   <!-- ur5 -->
-   <xacro:include filename="$(find ur_description)/urdf/ur5.urdf.xacro"/>
-   <!-- arm -->
-   <xacro:arg name="kinematics_config" default="$(find ur_description)/config/ur5_default.yaml"/>
-   <xacro:ur5_robot prefix="" joint_limited="true" shoulder_pan_lower_limit="${-pi}" shoulder_pan_upper_limit="${pi}" shoulder_lift_lower_limit="${-pi}" shoulder_lift_upper_limit="${pi}" elbow_joint_lower_limit="${-pi}" elbow_joint_upper_limit="${pi}" wrist_1_lower_limit="${-pi}" wrist_1_upper_limit="${pi}" wrist_2_lower_limit="${-pi}" wrist_2_upper_limit="${pi}" wrist_3_lower_limit="${-pi}" wrist_3_upper_limit="${pi}" transmission_hw_interface="$(arg transmission_hw_interface)" kinematics_file="${load_yaml('$(arg kinematics_config)')}"/>
-   <link name="world"/>
-   <joint name="world_joint" type="fixed">
-   <parent link="world"/>
-   <child link="base_link"/>
-   <origin xyz="0.0 0.0 0.0" rpy="0.0 0.0 0.0"/>
-   </joint>
+  <!-- common stuff -->
+  <xacro:include filename="$(find ur_description)/urdf/common.gazebo.xacro"/>
+  <!-- ur5 -->
+  <xacro:include filename="$(find ur_description)/urdf/ur5.urdf.xacro"/>
+  <!-- arm -->
+  <xacro:arg name="kinematics_config" default="$(find ur_description)/config/ur5_default.yaml"/>
+  <xacro:ur5_robot prefix="" joint_limited="true" shoulder_pan_lower_limit="${-pi}" shoulder_pan_upper_limit="${pi}" shoulder_lift_lower_limit="${-pi}" shoulder_lift_upper_limit="${pi}" elbow_joint_lower_limit="${-pi}" elbow_joint_upper_limit="${pi}" wrist_1_lower_limit="${-pi}" wrist_1_upper_limit="${pi}" wrist_2_lower_limit="${-pi}" wrist_2_upper_limit="${pi}" wrist_3_lower_limit="${-pi}" wrist_3_upper_limit="${pi}" transmission_hw_interface="$(arg transmission_hw_interface)" kinematics_file="${load_yaml('$(arg kinematics_config)')}"/>
+  <link name="world"/>
+  <joint name="world_joint" type="fixed">
+  <parent link="world"/>
+  <child link="base_link"/>
+  <origin xyz="0.0 0.0 0.0" rpy="0.0 0.0 0.0"/>
+  </joint>
   <link name="tool0_controller"/>
   <joint name="base_tool0_controller_floating_joint" type="fixed">

Commit message: druver update

File: lego_robot_description/urdf/lego_bot.xacro (robot description, xacro)
@@ -2,5 +2,6 @@
 <robot xmlns:xacro="http://wiki.ros.org/xacro"
        name="ur5" >
-   <xacro:arg name="transmission_hw_interface" default="hardware_interface/PositionJointInterface"/>
+  <link name="world"/>
+  <xacro:arg name="transmission_hw_interface" default="hardware_interface/PositionJointInterface"/>
   <!-- common stuff -->
   <xacro:include filename="$(find ur_description)/urdf/common.gazebo.xacro"/>
@@ -9,6 +10,5 @@
   <!-- arm -->
   <xacro:arg name="kinematics_config" default="$(find ur_description)/config/ur5_default.yaml"/>
-  <xacro:ur5_robot prefix="" joint_limited="true" shoulder_pan_lower_limit="${-pi}" shoulder_pan_upper_limit="${pi}" shoulder_lift_lower_limit="${-pi}" shoulder_lift_upper_limit="${pi}" elbow_joint_lower_limit="${-pi}" elbow_joint_upper_limit="${pi}" wrist_1_lower_limit="${-pi}" wrist_1_upper_limit="${pi}" wrist_2_lower_limit="${-pi}" wrist_2_upper_limit="${pi}" wrist_3_lower_limit="${-pi}" wrist_3_upper_limit="${pi}" transmission_hw_interface="$(arg transmission_hw_interface)" kinematics_file="${load_yaml('$(arg kinematics_config)')}"/>
-  <link name="world"/>
+  <xacro:ur5_robot prefix="" joint_limited="true" shoulder_pan_lower_limit="${0}" shoulder_pan_upper_limit="${2* pi}" shoulder_lift_lower_limit="${-pi}" shoulder_lift_upper_limit="${pi}" elbow_joint_lower_limit="${-pi}" elbow_joint_upper_limit="${pi}" wrist_1_lower_limit="${-pi}" wrist_1_upper_limit="${pi}" wrist_2_lower_limit="${-pi}" wrist_2_upper_limit="${pi}" wrist_3_lower_limit="${-pi}" wrist_3_upper_limit="${pi}" transmission_hw_interface="$(arg transmission_hw_interface)" kinematics_file="${load_yaml('$(arg kinematics_config)')}"/>
   <joint name="world_joint" type="fixed">
   <parent link="world"/>

File: lego_robot_description/urdf/table.xacro (robot description, xacro)
@@ -4,18 +4,4 @@
     <link
       name="table">
-      <inertial>
-        <origin
-          xyz="0.2005 -0.20049 -0.41445"
-          rpy="0 0 0" />
-        <mass
-          value="524.11" />
-        <inertia
-          ixx="54.974"
-          ixy="8.9479E-07"
-          ixz="-3.4714E-08"
-          iyy="54.792"
-          iyz="2.9131E-08"
-          izz="55.153" />
-      </inertial>
       <visual>
         <origin

Commit message: look into Rodrigues

File: lego_robot_description/urdf/lego_bot.xacro (robot description, xacro)
@@ -33,5 +33,5 @@
     <parent link="gripper_body" />
     <child link = "TCP" />
-    <origin xyz="0.0 -0.215 0.0" rpy="0.0 3.14159265359 3.14159265359" />
+    <origin xyz="0.0 -0.215 0.0" rpy="0.0 1.57079632679 -1.57079632679" />
   </joint>
   <!-- Realsense Cam -->

Commit message: rldy to go home

File: lego_robot_description/urdf/lego_bot.xacro (robot description, xacro)
@@ -33,5 +33,5 @@
     <parent link="gripper_body" />
     <child link = "TCP" />
-    <origin xyz="0.0 -0.215 0.0" rpy="0.0 1.57079632679 -1.57079632679" />
+    <origin xyz="0.0 -0.215 0.0" rpy="3.14159265359 1.57079632679 -1.57079632679" />
   </joint>
   <!-- Realsense Cam -->

Commit message: all done

File: lego_robot_description/urdf/lego_bot.xacro (robot description, xacro)
@@ -33,5 +33,5 @@
     <parent link="gripper_body" />
     <child link = "TCP" />
-    <origin xyz="0.0 -0.215 0.0" rpy="3.14159265359 1.57079632679 -1.57079632679" />
+    <origin xyz="0.0 -0.233 -0.01905" rpy="3.14159265359 1.57079632679 -1.57079632679" />
   </joint>
   <!-- Realsense Cam -->
